Commit message: policy upload

File: rsc/pogo/urdf/pogo.urdf (robot description, URDF)
Before this commit: robot pogo, 7 links, 6 joints
Joints:
- joint guide_mass: limit lower=0 upper=0.4 effort=3500 -> lower=0 upper=0.4 effort=1750

Commit message: curriculum change

File: rsc/pogo/urdf/pogo.urdf (robot description, URDF)
Before this commit: robot pogo, 7 links, 6 joints
Joints:
- joint guide_mass: limit lower=0 upper=0.4 effort=1750 -> lower=0 upper=0.4 effort=1750 velocity=4.0

Commit message: minor changes

File: rsc/pogo/urdf/pogo.urdf (robot description, URDF)
Before this commit: robot pogo, 7 links, 6 joints
Joints:
- joint base_cross: limit lower=-1.0472 upper=1.0472 effort=700 -> lower=-0.523599 upper=0.523599 effort=350 velocity=1.0
- joint cross_guide: limit lower=-1.0472 upper=1.0472 effort=700 -> lower=-0.523599 upper=0.523599 effort=350 velocity=1.0
- joint guide_mass: limit lower=0 upper=0.4 effort=1750 velocity=4.0 -> lower=0 upper=0.3 effort=1750 velocity=4.0

Commit message: successful pogostick! code & policy upload

File: rsc/pogo/urdf/pogo.urdf (robot description, URDF)
Before this commit: robot pogo, 7 links, 6 joints
Joints:
- joint base_cross: limit lower=-0.523599 upper=0.523599 effort=350 velocity=1.0 -> lower=-0.4 upper=0.4 effort=1000 velocity=4.0
- joint cross_guide: limit lower=-0.523599 upper=0.523599 effort=350 velocity=1.0 -> lower=-0.4 upper=0.4 effort=1000 velocity=4.0
- joint guide_mass: limit lower=0 upper=0.3 effort=1750 velocity=4.0 -> lower=0 upper=0.3 effort=2100 velocity=4.0
